Commit message: test commit

File: description/robot_core.xacro (robot description, xacro)
@@ -20,5 +20,5 @@
         <origin xyz="-0.1 0 0"/>
     </joint>
-    <link name+"chassis">
+    <link name="chassis">
         <visual>
             <origin xyz="0.15 0 0.075" rpy="0 0 0" />

Commit message: test commit

File: description/robot_core.xacro (robot description, xacro)
@@ -1,5 +1,4 @@
 <?xml version="1.0"?>
 <robot xmlns:xacro="http://www.ros.org/wiki/xacro" >
-<<<<<<< HEAD
     <material name="white">
         <color rgba="1 1 1 1" />
@@ -31,33 +30,2 @@
     </link>
 </robot>
-=======
-    <material name="white">
-        <color rgba="1 1 1 1" />
-    </material>
-    <material name="orange">
-        <color rgba="1 0.3 0.1 1" />
-    </material>
-    <material name="blue">
-        <color rgba="0.2 0.2 1 1" />
-    </material>
-    <material name="black">
-        <color rgba="0 0 0 1" />
-    </material>
-    <link name="base_link">
-    </link>
-    <joint name="chassis_joint" type="fixed">
-        <parent link="base_link"/>
-        <child link="chassis"/>
-        <origin xyz="-0.1 0 0"/>
-    </joint>
-    <link name="chassis">
-        <visual>
-            <origin xyz="0.15 0 0.075" rpy="0 0 0" />
-            <geometry>
-                <box size="0.3 0.3 0.15"/>
-            </geometry>
-            <material name="white"/>
-        </visual>
-    </link>
-</robot>
->>>>>>> 5fe40e682cd30fb0c81a241842da96493a9382f7

Commit message: test commit

File: description/robot_core.xacro (robot description, xacro)
@@ -13,6 +13,8 @@
         <color rgba="0 0 0 1" />
     </material>
+    <!-- BASE LINK-->
     <link name="base_link">
     </link>
+    <!-- CHASSIS LINK-->
     <joint name="chassis_joint" type="fixed">
         <parent link="base_link" />
@@ -29,3 +31,33 @@
         </visual>
     </link>
+<!-- LEFT WHEEL LINK-->
+    <joint name="left_wheel_joint" type="continuous">
+        <parent link="base_link"/>
+        <child link="left_wheel"/>
+        <origin xyz="0 0.175 0" rpy="-${pi/2} 0 0"/>
+        <axis xyz="0 0 1"/>
+    </joint>
+    <link name="left_wheel">
+        <visual>
+            <geometry>
+                <cylinder radius="0.05" length="0.04"/>
+            </geometry>
+            <material name="blue"/>
+        </visual>
+    </link>
+ <!--RIGHT WHEEL LINK-->
+    <joint name="right_wheel_joint" type="continuous">
+        <parent link="base_link"/>
+        <child link="right_wheel"/>
+        <origin xyz="0 0.175 0" rpy="${pi/2} 0 0"/>
+        <axis xyz="0 0 -1"/>
+    </joint>
+    <link name="right_wheel">
+        <visual>
+            <geometry>
+                <cylinder radius="0.05" length="0.04"/>
+            </geometry>
+            <material name="blue"/>
+        </visual>
+    </link>
 </robot>
